File: USB-C-3-way-splitter.kicad_pcb (KiCad board)
At the start: 2 copper layers, 29 x 27 mm, 35 parts, among them J1 USB_C_Receptacle_USB2.0, J2 Conn_01x04, J3 Conn_01x04, J4 Conn_01x04, U1 LM393, U2 SiP32509

Commit message: Updated design files for V2
Other:
- board text added: "+5V"
- board text added: "D+"
- board text added: "D-"
- board text added: "GND"
- board text added: "JLCJLCJLCJLC"
- board text added: "Note the output connector pads for +5V and GND have enlarged holes and pads."
Changed lines of the file:
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@@
 		(tags "fuse handsolder")
 		(property "Reference" "F1"
-			(at 0 -2.65 270)
+			(at 0 -2.65 -90)
 			(layer "F.SilkS")
 			(effects
@@
 		)
 		(fp_text user "${REFERENCE}"
-			(at 0 0 270)
+			(at 0 0 -90)
 			(layer "F.Fab")
 			(effects
@@
 			(at 0 0)
 			(size 1.35 1.35)
-			(drill 0.8)
+			(drill 1)
 			(layers "*.Cu" "*.Mask")
 			(remove_unused_layers no)
@@
 			(pintype "passive")
 		)
-		(pad "4" thru_hole oval
+		(pad "4" thru_hole circle
 			(at 0 6)
-			(size 1.35 1.35)
-			(drill 0.8)
+			(size 1.5 1.5)
+			(drill 1)
 			(layers "*.Cu" "*.Mask")
 			(remove_unused_layers no)
@@
 		)
 		(model "${KICAD8_3DMODEL_DIR}/Connector_PinHeader_2.00mm.3dshapes/PinHeader_1x04_P2.00mm_Vertical.wrl"
+			(hide yes)
 			(offset
 				(xyz 0 0 0)
@@
 		(tags "SOIC SO")
 		(property "Reference" "U1"
-			(at -1.45 3.45 360)
+			(at -1.45 3.45 0)
 			(layer "F.SilkS")
 			(effects
@@
 		)
 		(property "Value" "LM393"
-			(at 0 3.4 360)
+			(at 0 3.4 0)
 			(layer "F.Fab")
 			(effects
@@
 		)
 		(fp_text user "${REFERENCE}"
-			(at 0 0 360)
+			(at 0 0 0)
 			(layer "F.Fab")
 			(effects
@@
 		)
 		(property "Value" "22uF"
-			(at 0 1.85 270)
+			(at 0 1.85 -90)
 			(layer "F.Fab")
 			(effects
@@
 		)
 		(fp_text user "${REFERENCE}"
-			(at 0 0 270)
+			(at 0 0 -90)
 			(layer "F.Fab")
 			(effects
@@
 		)
 		(property "Value" "LED"
-			(at 0 1.65 270)
+			(at 0 1.65 -90)
 			(layer "F.Fab")
 			(effects
@@
 		)
 		(fp_text user "${REFERENCE}"
-			(at 0 0 270)
+			(at 0 0 -90)
 			(layer "F.Fab")
 			(effects
@@
 		(tags "LED handsolder")
 		(property "Reference" "D3"
-			(at -0.15 -1.6 270)
+			(at -0.15 -1.6 -90)
 			(layer "F.SilkS")
 			(effects
@@
 		)
 		(property "Value" "LED"
-			(at 0 1.65 270)
+			(at 0 1.65 -90)
 			(layer "F.Fab")
 			(effects
@@
 		)
 		(fp_text user "${REFERENCE}"
-			(at 0 0 270)
+			(at 0 0 -90)
 			(layer "F.Fab")
 			(effects
@@
 		(pad "1" thru_hole rect
 			(at 0 0)
-			(size 1.35 1.35)
-			(drill 0.8)
+			(size 1.5 1.5)
+			(drill 1)
 			(layers "*.Cu" "*.Mask")
 			(remove_unused_layers no)
@@
 		(pad "4" thru_hole oval
 			(at 0 6)
-			(size 1.35 1.35)
-			(drill 0.8)
+			(size 1.5 1.5)
+			(drill 1)
 			(layers "*.Cu" "*.Mask")
 			(remove_unused_layers no)
@@
 		)
 		(model "${KICAD8_3DMODEL_DIR}/Connector_PinHeader_2.00mm.3dshapes/PinHeader_1x04_P2.00mm_Vertical.wrl"
+			(hide yes)
 			(offset
 				(xyz 0 0 0)
@@
 		)
 		(fp_text user "${REFERENCE}"
-			(at 0 0 270)
+			(at 0 0 -90)
 			(layer "F.Fab")
 			(effects
@@
 		)
 		(property "Value" "100"
-			(at 0 1.65 270)
+			(at 0 1.65 -90)
 			(layer "F.Fab")
 			(effects
@@
 		)
 		(fp_text user "${REFERENCE}"
-			(at 0 0 270)
+			(at 0 0 -90)
 			(layer "F.Fab")
 			(effects
@@
 		)
 		(property "Value" "4.7uF"
-			(at 0 1.68 270)
+			(at 0 1.68 -90)
 			(layer "F.Fab")
 			(effects
@@
 		)
 		(fp_text user "${REFERENCE}"
-			(at 0 0 270)
+			(at 0 0 -90)
 			(layer "F.Fab")
 			(effects
@@
 		)
 		(property "Value" "100"
-			(at 0 1.65 270)
+			(at 0 1.65 -90)
 			(layer "F.Fab")
 			(effects
@@
 		)
 		(fp_text user "${REFERENCE}"
-			(at 0 0 270)
+			(at 0 0 -90)
 			(layer "F.Fab")
 			(effects
@@
 		(pad "1" thru_hole rect
 			(at 0 0)
-			(size 1.35 1.35)
-			(drill 0.8)
+			(size 1.5 1.5)
+			(drill 1)
 			(layers "*.Cu" "*.Mask")
 			(remove_unused_layers no)
@@
 			(pintype "passive")
 		)
-		(pad "4" thru_hole oval
+		(pad "4" thru_hole circle
 			(at 0 6)
-			(size 1.35 1.35)
-			(drill 0.8)
+			(size 1.5 1.5)
+			(drill 1)
 			(layers "*.Cu" "*.Mask")
 			(remove_unused_layers no)
@@
 		)
 		(model "${KICAD8_3DMODEL_DIR}/Connector_PinHeader_2.00mm.3dshapes/PinHeader_1x04_P2.00mm_Vertical.wrl"
+			(hide yes)
 			(offset
 				(xyz 0 0 0)
@@
 		(tags "test point SMD pad")
 		(property "Reference" "TP3"
-			(at 0 2.148 180)
+			(at 0.55 2.3 180)
 			(layer "B.SilkS")
 			(effects
@@
 		(layer "Edge.Cuts")
 	)
+	(gr_text "+5V"
+		(at 25.1 -2.3 0)
+		(layer "B.SilkS")
+		(effects
+			(font
+				(size 1.2 1.2)
+				(thickness 0.15)
+			)
+			(justify left bottom mirror)
+		)
+	)
 	(gr_text "EN"
-		(at 21.85 2.75 0)
+		(at 21.6 2.45 0)
 		(layer "B.SilkS")
 		(effects
@@
 		)
 	)
+	(gr_text "JLCJLCJLCJLC"
+		(at 17 -12 0)
+		(layer "B.SilkS")
+		(effects
+			(font
+				(size 1 1)
+				(thickness 0.15)
+			)
+			(justify left bottom mirror)
+		)
+	)
 	(gr_text "USB-C Splitter V2\nPylon April 13 24"
 		(at 17.1 -8.55 90)
@@
 	)
 	(gr_text "CC2"
-		(at 13.85 3.6 0)
+		(at 13.55 3.25 0)
 		(layer "B.SilkS")
 		(effects
@@
 	)
 	(gr_text "+1.2V"
-		(at 13.75 12.65 0)
+		(at 15.05 13.3 0)
 		(layer "B.SilkS")
 		(effects
@@
 		)
 	)
+	(gr_text "D+"
+		(at 25.15 -0.25 0)
+		(layer "B.SilkS")
+		(effects
+			(font
+				(size 1.2 1.2)
+				(thickness 0.15)
+			)
+			(justify left bottom mirror)
+		)
+	)
+	(gr_text "D-"
+		(at 25.15 1.75 0)
+		(layer "B.SilkS")
+		(effects
+			(font
+				(size 1.2 1.2)
+				(thickness 0.15)
+			)
+			(justify left bottom mirror)
+		)
+	)
+	(gr_text "GND"
+		(at 25.15 3.75 0)
+		(layer "B.SilkS")
+		(effects
+			(font
+				(size 1.2 1.2)
+				(thickness 0.15)
+			)
+			(justify left bottom mirror)
+		)
+	)
+	(gr_text "Note the output connector pads for +5V and GND have enlarged holes and pads."
+		(at 30 -9 0)
+		(layer "Cmts.User")
+		(effects
+			(font
+				(size 1 1)
+				(thickness 0.15)
+			)
+			(justify left bottom)
+		)
+	)
 	(segment
 		(start 8.525 3.805)
@@
 		(polygon
 			(pts
-				(xy -1.2 -6.9) (xy 5.2 -6.9) (xy 5.2 6.7) (xy -1.2 6.7)
+				(xy -1.2 -13.9) (xy 5.2 -13.9) (xy 5.2 13.7) (xy -1.2 13.7)
 			)
 		)
