File: USB-C-3-way-splitter.kicad_pcb (KiCad board)
At the start: 2 copper layers, 29 x 27 mm, 35 parts, among them J1 USB_C_Receptacle_USB2.0, J2 Conn_01x04, J3 Conn_01x04, J4 Conn_01x04, U1 LM393, U2 SiP32509

Commit message: Some organization and updates
Parts:
- added D6: D_Zener, Diode_SMD:D_SOD-523, F.Cu at (23.2, -6.50)
- added U3: SRV05-4, Package_TO_SOT_SMD:SOT-23-6, F.Cu at (8.20, 9.00)
- R3: value 4.7K -> 4.7k
- R4, R5: value 100 -> 470
- moved R1 6.13 mm to (10.5, 12.1), turned to 0 degrees
- moved C5 4.18 mm to (14.5, 11.0), turned to 0 degrees
- moved R2 2.40 mm to (11.5, 9.00)
- moved TP2 0.51 mm to (7.80, 3.50)
- moved H7 0.50 mm to (23.5, 12.0)
- moved TP1 0.40 mm to (7.60, -0.50)
- moved D2 0.10 mm to (8.20, -9.22)
Connections:
- net Net-(F1-Pad1) renamed V-UNFUSED
Routing:
- net V-UNFUSED: track 11.3 -> 20.6 mm
- net CC1: track 13.9 -> 21.2 mm, vias 1 -> 3
- net CC2: track 15.3 -> 20.8 mm
- net +1V2: track 19.5 -> 20.4 mm
- net GND: vias 12 -> 20
Other:
- board text added: "IN OK"
- board text added: "OUT OK"
- board text added: "USB-C Splitter V3 Pylon May 7 2024 5V 3A in 3x 5V 1A out"
- board text removed: "USB-C Splitter V2 Pylon April 13 24"
