File: USB-C-3-way-splitter.kicad_sch (KiCad schematic)
At the start: 35 parts, among them J1 USB_C_Receptacle_USB2.0, J2 Conn_01x04, J3 Conn_01x04, J4 Conn_01x04, U1 LM393, U2 SiP32509

Commit message: Updated design files for V2
Parts:
- R3: value 4.7K -> 4.7k
- R4, R5: value 100 -> 470
Changed lines of the file:
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@@
 		(fields_autoplaced yes)
 		(property "Reference" "R4"
-			(at 58.42 88.9 0)
-			(effects
-				(font
-					(size 1.27 1.27)
-				)
-				(justify left)
-			)
-		)
-		(property "Value" "100"
-			(at 58.42 91.44 0)
+			(at 58.42 88.8999 0)
+			(effects
+				(font
+					(size 1.27 1.27)
+				)
+				(justify left)
+			)
+		)
+		(property "Value" "470"
+			(at 58.42 91.4399 0)
 			(effects
 				(font
@@
 		(fields_autoplaced yes)
 		(property "Reference" "R8"
-			(at 153.67 105.41 0)
+			(at 153.67 105.4099 0)
 			(effects
 				(font
@@
 		)
 		(property "Value" "1k"
-			(at 153.67 107.95 0)
+			(at 153.67 107.9499 0)
 			(effects
 				(font
@@
 		(fields_autoplaced yes)
 		(property "Reference" "R6"
-			(at 153.67 80.01 0)
+			(at 153.67 80.0099 0)
 			(effects
 				(font
@@
 		)
 		(property "Value" "1k"
-			(at 153.67 82.55 0)
+			(at 153.67 82.5499 0)
 			(effects
 				(font
@@
 			)
 		)
-		(property "Value" "4.7K"
+		(property "Value" "4.7k"
 			(at 104.14 88.9 0)
 			(effects
@@
 		(fields_autoplaced yes)
 		(property "Reference" "R5"
-			(at 69.85 88.9 0)
-			(effects
-				(font
-					(size 1.27 1.27)
-				)
-				(justify left)
-			)
-		)
-		(property "Value" "100"
-			(at 69.85 91.44 0)
-			(effects
-				(font
+			(at 69.85 88.8999 0)
+			(effects
+				(font
+					(size 1.27 1.27)
+				)
+				(justify left)
+			)
+		)
+		(property "Value" "470"
+			(at 69.85 91.4399 0)
+			(effects
+				(font

Commit message: Some organization and updates
Parts:
- added D6: D_Zener, Diode_SMD:D_SOD-523, symbol Device:D_Zener
- added U3: SRV05-4, Package_TO_SOT_SMD:SOT-23-6, symbol Power_Protection:SRV05-4
Connections:
- net +5V: now also D6.1 (K)
- net CC1: now also U3.3 (IO2)
- net CC2: now also U3.4 (IO3)
- net GND: now also D6.2 (A), U3.2 (VN)
- net V-UNFUSED: now reaches F1.1, J1.A4 (VBUS), J1.A9 (VBUS), J1.B4 (VBUS), J1.B9 (VBUS)
- net V-UNFUSED: now also U3.5 (VP)
Other:
- note added: "ESD protection"
- note added: "ESD5Z5V0"
- moved on the sheet: C1, C2, C3, C5, D1, D2, D3, D4, D5, F1, J1, J2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
