File: V4/USB-C-3-way-splitter-V4.kicad_pcb (KiCad board)
At the start: 2 copper layers, 29 x 27 mm, 33 parts, among them J1 USB_C_Receptacle_USB2.0, J2 Conn_01x04, J3 Conn_01x04, J4 Conn_01x04, U1 LM393, U3 SRV05-4

Commit message: More work on V4
Parts:
- added C2: 22uF, Capacitor_SMD:C_1206_3216Metric_Pad1.33x1.80mm_HandSolder, F.Cu at (21.9, 2.50)
- added D4: 1N4148W, Diode_SMD:D_SOD-123, F.Cu at (13.1, -6.90)
- added D5: 1N4148W, Diode_SMD:D_SOD-123, F.Cu at (13.9, -3.30)
- added Q1: 2N7002, Package_TO_SOT_SMD:SOT-23, F.Cu at (17.2, -4.00)
- added R8: 1k, Resistor_SMD:R_0805_2012Metric_Pad1.20x1.40mm_HandSolder, F.Cu at (11.7, -2.80)
- added R9: 1k, Resistor_SMD:R_0805_2012Metric_Pad1.20x1.40mm_HandSolder, F.Cu at (17.8, 0.40)
- moved R6 5.36 mm to (17.1, 5.00)
- moved R4 2.80 mm to (7.40, -9.30)
- moved D2 2.36 mm to (9.50, -11.2), turned to -90 degrees
- moved C3 1.11 mm to (11.8, -10.6)
- moved D3 0.91 mm to (20.1, 4.70), turned to 0 degrees
- moved C1 0.82 mm to (20.2, -0.76)
- moved R7 0.82 mm to (22.3, -0.80)
- moved U2 0.46 mm to (21.4, -4.46)
- moved F1 0.40 mm to (8.70, -4.08)
- moved D6 0.28 mm to (23.4, -6.70), turned to 90 degrees
Connections:
- U1 pad 1: EN-OPEN-COL -> Net-(D4-A)
- U1 pad 7: EN-OPEN-COL -> Net-(D5-A)
Routing:
- net Net-(D5-A): track 0.00 -> 11.8 mm, vias 0 -> 2
- net Net-(D4-A): track 0.00 -> 11.7 mm, vias 0 -> 2
- net EN-OPEN-COL: track 18.2 -> 9.35 mm
- net VBUS: track 2.37 -> 9.44 mm
- net Net-(U2-SENSE): track 4.10 -> 10.0 mm
- net Net-(D4-K): track 0.00 -> 4.21 mm
- net GND: vias 18 -> 19
Other:
- board text removed: "IN OK"
- board text removed: "OUT OK"
