File: V4/USB-C-3-way-splitter-V4.kicad_sch (KiCad schematic)
At the start: 33 parts, among them J1 USB_C_Receptacle_USB2.0, J2 Conn_01x04, J3 Conn_01x04, J4 Conn_01x04, U1 LM393, U3 SRV05-4

Commit message: More work on V4
Parts:
- added C2: 22uF, Capacitor_SMD:C_1206_3216Metric_Pad1.33x1.80mm_HandSolder, symbol Device:C
- added D4, D5: 1N4148W, Diode_SMD:D_SOD-123, symbol Diode:1N4148W
- added Q1: 2N7002, Package_TO_SOT_SMD:SOT-23, symbol Transistor_FET:2N7002
- added R8, R9: 1k, Resistor_SMD:R_0805_2012Metric_Pad1.20x1.40mm_HandSolder, symbol Device:R
Connections:
- net +5V: now also C2.1
- net EN-OPEN-COL: now also Q1.3 (D); no longer U1.1, U1.7
- net GND: now also C2.2, Q1.2 (S)
- net VBUS: now also R8.1, R9.1
- new net: D4.1 (K), D5.1 (K), Q1.1 (G)
- new net: D5.2 (A), R9.2, U1.7
- new net: D4.2 (A), R8.2, U1.1
Other:
- note added: "NIS6452MT1TWG"
- moved on the sheet: C3
